File: Hardware/SparkFun_Qwiic_Relay_1x1A_DPDT/SparkFun_Qwiic_Relay_1x1A_DPDT.kicad_sch (KiCad schematic)
At the start: 36 parts, among them J1 Qwiic_RA, J2 Conn_01x03, J3 Qwiic_RA, J4 Conn_01x01, J5 I2C, J6 3.5mm, K2 G6K-2F-Y DC3, Q2 LMUN2235LT1G, U1 PCA9536DP, U3 EL3H7

Commit message: Post review update
Parts:
- removed U1: PCA9536DP, SparkFun-Semiconductor-Standard:TSSOP-8_3x3mm_P0.65mm, symbol SparkFun-IC-Special-Function:PCA9536DP
- added JP1: ADR, SparkFun-Jumper:Jumper_2_NO, symbol SparkFun-Jumper:SolderJumper_2_Open
- added R3: 10k, SparkFun-Resistor:R_0603_1608Metric, symbol SparkFun-Resistor:10k_0603
- added U2: TCA9555RTWR, SparkFun-Semiconductor-Standard:QFN-24-1EP_4x4mm_P0.5mm_EP2.45x2.45mm, symbol SparkFun-IC-Special-Function:TCA9555RTWR
- JP4: value ~ -> LED
Connections:
- net 3.3V: now also JP1.2 (B), U2.21 (VCC)
- net GND: now also R3.1, U2.23 (A1), U2.24 (A2), U2.25 (EPAD), U2.9 (GND)
- net I2C_Drive: now also U2.1 (P00)
- net IO2: now also U2.3 (P02)
- net IO3: now also U2.4 (P03)
- net SCL: now also U2.19 (SCL)
- net SDA: now also U2.20 (SDA)
- net STAT_LED: now also U2.2 (P01)
- new net: JP1.1 (A), R3.2, U2.18 (A0)
Other:
- note added: "Close ADR for 0x21"
- note added: "Default 7-bit Unshifted I²C Address: 0x20"
- note added: "Extra I/O"
- note added: "TCA9555RTWR(UMW) - QFN-24 (4x4) drop in for TCA. Cheapest. UMW brand. PI4IOE5V9535ZDEX - QFN-24 (4x4) drop in for TCA. Diode brand. TCA9555RTWR - WQFN-24 (4x4) 0x20 as default adr. TI watermark. XL9555QF24 - QFN-24 (4x4) drop in for TCA. AW9523BTQR - TQFN-24 (4x4) Very good but has RST, for A1. 0x51 as default. XL9535QF24 - QFN-24 (4x4) PCA9536DGKR - VSSOP-8 TCA9537DGSR - MSOP-10"
- note removed: "Default 7-bit Unshifted I²C Address: 0x41"
- note removed: "Unused I/O"
- moved on the sheet: C1

Commit message: Adds prod-id to 16-bit IO Expander
Parts:
- U2: PROD_ID IC-... -> IC-27579
Changed lines of the file:
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@@
 			)
 		)
-		(property "PROD_ID" "IC-..."
+		(property "PROD_ID" "IC-27579"
 			(at 87.63 100.33 0)
 			(effects
